Commit message: Modified camera urdf
Signed-off-by: kijonggil <kkjong@robotis.com>

File: turtlebot3_description/urdf/turtlebot3_burger_camera.urdf (robot description, URDF)
Before this commit: robot turtlebot3_burger, 10 links, 9 joints
Joints:
- joint camera_joint: origin xyz=0.040 -0.011 0.130 rpy=0 0.174 0 -> xyz=0.040 -0.011 0.130 rpy=0 0 0
